File: PCB/herringbone_macro_pad.kicad_pcb (KiCad board)
At the start: 2 copper layers, 114.3 x 114.3 mm, 33 parts, among them J1 Screw_Terminal_01x04, SW1 CherryMX_2.75u_PCB_StabWireBo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, SW10 CherryMX_1.00u_PCB, SW11 SW_Push, SW2 CherryMX_1.00u_PCB, SW3 CherryMX_2.75u_PCB_StabWireBo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, SW4 CherryMX_2.75u_PCB_StabWireBo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, SW5 CherryMX_1.00u_PCB, SW6 CherryMX_2.75u_PCB_StabWireBo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, SW7 CherryMX_2.75u_PCB_StabWireBo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

Commit message: Hardware revision.
Parts:
- removed R5: 10k, Keebio-Parts:R_0603
- added C13: 0.1u, Keebio-Parts:C_0402, F.Cu at (196.7, 64.6)
- added C14: 0.1u, Keebio-Parts:C_0402, F.Cu at (171.8, 111.0)
- added C15: 0.1u, Keebio-Parts:C_0402, F.Cu at (170.1, 109.0)
- added R3: 10k, Keebio-Parts:R_0402, F.Cu at (136.3, 106.7)
- added SW12: CherryMX_2.75u_PCB_StabWireBottom, Button_Switch_Keyboard:SW_Cherry_MX_2.75u_PCB, B.Cu at (116.5, 102.1)
- C1: value 22p -> 22u; footprint Keebio-Parts:C_0603 -> Keebio-Parts:C_0402; moved to F.Cu
- C10: value 10n -> 0.1u; footprint Keebio-Parts:C_0603 -> Keebio-Parts:C_0402; moved to F.Cu
- C11: value 1u -> 30p; footprint Keebio-Parts:C_0603 -> Keebio-Parts:C_0402; moved to F.Cu
- C12: value 0.1u -> 30p; footprint Keebio-Parts:C_0603 -> Keebio-Parts:C_0402; moved to F.Cu
- C2: value 22p -> 10u; footprint Keebio-Parts:C_0603 -> Keebio-Parts:C_0402; moved to F.Cu
- C3: value 22u -> 4.7u; footprint Keebio-Parts:C_0603 -> Keebio-Parts:C_0402; moved to F.Cu
- C4: value 10u -> 4.7u; footprint Keebio-Parts:C_0603 -> Keebio-Parts:C_0402; moved to F.Cu
- C5: value 4.7u -> 0.1u; footprint Keebio-Parts:C_0603 -> Keebio-Parts:C_0402; moved to F.Cu
- C6, C7, C9: value 100n -> 0.1u; footprint Keebio-Parts:C_0603 -> Keebio-Parts:C_0402; moved to F.Cu
- C8: value 100n -> 4.7u; footprint Keebio-Parts:C_0603 -> Keebio-Parts:C_0402; moved to F.Cu
- D1, U1, U2, USB1, Y1: moved to F.Cu
- J1: value Screw_Terminal_01x04 -> JST; moved to F.Cu
- R1, R2: footprint Keebio-Parts:R_0603 -> Keebio-Parts:R_0402; moved to F.Cu
- SW1: value CherryMX_2.75u_PCB_StabWireBottom -> SW_Push; footprint CherryMX_PCB_StabWireBottom:CherryMX_2.75u_PCB_StabWireBottom -> Keebio-Parts:SW_SPST_TL3342
- SW10, SW5: value CherryMX_1.00u_PCB -> CherryMX_2.75u_PCB_StabWireBottom; footprint CherryMX_PCB:CherryMX_1.00u_PCB -> Button_Switch_Keyboard:SW_Cherry_MX_2.75u_PCB; moved to B.Cu
- SW11: value SW_Push -> CherryMX_1.00u_PCB; footprint Keebio-Parts:SW_SPST_TL3342 -> Button_Switch_Keyboard:SW_Cherry_MX_1.00u_PCB
- SW2: value CherryMX_1.00u_PCB -> SW_SPST; footprint CherryMX_PCB:CherryMX_1.00u_PCB -> Button_Switch_SMD:SW_SPDT_PCM12
- SW3, SW6, SW7: footprint CherryMX_PCB_StabWireBottom:CherryMX_2.75u_PCB_StabWireBottom -> Button_Switch_Keyboard:SW_Cherry_MX_2.75u_PCB; moved to B.Cu
- SW4, SW9: value CherryMX_2.75u_PCB_StabWireBottom -> CherryMX_1.00u_PCB; footprint CherryMX_PCB_StabWireBottom:CherryMX_2.75u_PCB_StabWireBottom -> Button_Switch_Keyboard:SW_Cherry_MX_1.00u_PCB; moved to B.Cu
- SW8: footprint CherryMX_PCB:CherryMX_1.00u_PCB -> Button_Switch_Keyboard:SW_Cherry_MX_1.00u_PCB; moved to B.Cu
- U3: value STM32L151C8TxA -> STM32F411CEUx; footprint Package_QFP:LQFP-48_7x7mm_P0.5mm -> Package_DFN_QFN:QFN-48-1EP_7x7mm_P0.5mm_EP5.6x5.6mm; moved to F.Cu
- moved SW10 76.0 mm to (149.7, 74.0), turned to -90 degrees
- moved SW6 63.9 mm to (135.6, 121.1), turned to 180 degrees
- moved SW9 53.9 mm to (187.8, 147.8), turned to -90 degrees
- moved C6 50.9 mm to (164.0, 118.3), turned to 0 degrees
- moved SW5 47.9 mm to (154.6, 140.2), turned to 180 degrees
- moved SW11 42.2 mm to (171.3, 121.1), turned to 180 degrees
- moved C5 37.8 mm to (196.5, 69.4)
- moved C7 37.7 mm to (196.5, 70.6)
- moved SW3 36.5 mm to (168.8, 93.0), turned to -90 degrees
- moved SW2 36.4 mm to (139.0, 110.0), turned to 0 degrees
- moved U2 36.1 mm to (192.9, 90.2), turned to 180 degrees
- moved C10 35.4 mm to (194.7, 77.7), turned to 0 degrees
- moved SW8 31.4 mm to (149.7, 109.7), turned to -90 degrees
- moved SW4 31.3 mm to (133.2, 83.0), turned to 180 degrees
- moved SW7 30.1 mm to (187.8, 112.1), turned to -90 degrees
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Connections:
- net /SW_8 renamed SW_3
- net /SW_9 renamed SW_4
- C1 pad 1: GND -> +5V
- C1 pad 2: /CLK_IN -> GND
- C11 pad 1: +3.3VA -> GND
- C11 pad 2: GND -> /CLK_IN
- C12 pad 1: /RST -> /CLK_OUT
- C2 pad 1: /CLK_OUT -> Net-(C2-Pad1)
- C3 pad 1: +5V -> +3.3VA
- C4 pad 1: Net-(C4-Pad1) -> +3.3VA
- C8 pad 1: +3.3VA -> /V_CAP
- SW1 pad 1: /SW_0 -> /RST
- SW11 pad 1: /RST -> SW_10
- SW2 pad 1: /SW_5 -> Net-(R3-Pad2)
- SW2 pad 2: GND -> /BOOT
- SW3 pad 1: /SW_1 -> SW_1
- SW4 pad 1: /SW_6 -> SW_6
- SW5 pad 1: /SW_2 -> SW_7
- SW6 pad 1: /SW_7 -> SW_2
- SW7 pad 1: /SW_3 -> SW_8
- SW9 pad 1: /SW_4 -> SW_9
- U2 pad 1: Net-(C4-Pad1) -> Net-(C2-Pad1)
- U3 pad 17: /SW_2 -> unconnected-(U3-Pad17)
- U3 pad 18: /SW_3 -> SW_1
- U3 pad 19: /SW_6 -> SW_5
- U3 pad 20: /SW_0 -> SW_2
- U3 pad 21: /SW_5 -> unconnected-(U3-Pad21)
- U3 pad 22: /SW_1 -> /V_CAP
- U3 pad 37: /SW_7 -> unconnected-(U3-Pad37)
- U3 pad 38: /SW_4 -> unconnected-(U3-Pad38)
- U3 pad 41: unconnected-(U3-Pad41) -> SW_6
- U3 pad 42: unconnected-(U3-Pad42) -> SW_7
- U3 pad 43: unconnected-(U3-Pad43) -> SW_10
- U3 pad 44: unconnected-(U3-Pad44) -> /BOOT
- U3 pad 45: unconnected-(U3-Pad45) -> SW_9
- U3 pad 46: unconnected-(U3-Pad46) -> SW_8
Routing:
- net SW_4: track 67.8 -> 0.00 mm
- net +3.3VA: track 66.7 -> 0.00 mm, vias 2 -> 0
- net /SW_3: track 61.2 -> 0.00 mm
- net +5V: track 51.8 -> 0.00 mm, vias 4 -> 0
- net SW_3: track 46.4 -> 0.00 mm
- net /SW_0: track 44.0 -> 0.00 mm
- net /SW_6: track 43.3 -> 0.00 mm
- net /D1-: track 47.0 -> 3.91 mm, vias 2 -> 0
- net /SW_4: track 40.7 -> 0.00 mm
- net /D1+: track 43.2 -> 3.93 mm
- net /SW_1: track 30.2 -> 0.00 mm
- net /RST: track 12.6 -> 40.1 mm
- net /SW_2: track 21.2 -> 0.00 mm
- net /SW_5: track 21.0 -> 0.00 mm
- net /SW_7: track 13.4 -> 0.00 mm
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Other:
- board outline removed

Commit message: Hardware revision 2/17/2022
Parts:
- added D2: LED, Diode_SMD:D_0402_1005Metric, F.Cu at (192.9, 96.4)
- added R4: 370, Keebio-Parts:R_0402, F.Cu at (192.8, 95.2)
- moved C13 47.4 mm to (151.8, 79.7), turned to -90 degrees
- moved C5 42.4 mm to (155.4, 79.7), turned to -90 degrees
- moved C10 41.7 mm to (153.0, 79.7), turned to 90 degrees
- moved C6 41.3 mm to (149.4, 79.7), turned to 90 degrees
- moved C7 40.9 mm to (156.6, 79.7), turned to -90 degrees
- moved C4 39.5 mm to (157.8, 79.7), turned to 90 degrees
- moved C3 38.1 mm to (159.0, 79.7), turned to 90 degrees
- moved C14 37.9 mm to (150.6, 79.7), turned to -90 degrees
- moved C9 35.2 mm to (154.2, 79.7), turned to 90 degrees
- moved C15 30.3 mm to (142.1, 97.6), turned to 90 degrees
- moved C2 24.6 mm to (186.4, 87.3), turned to 90 degrees
- moved C1 23.6 mm to (186.9, 89.3), turned to 180 degrees
- moved D1 19.0 mm to (185.3, 91.5), turned to -90 degrees
- moved U1 1.89 mm to (154.8, 59.6)
- moved R1 1.73 mm to (156.9, 56.1), turned to 180 degrees
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Connections:
- C1 pad 1: +5V -> +3.3VA
- U3 pad 17: unconnected-(U3-Pad17) -> SW_10
- U3 pad 18: SW_1 -> SW_9
- U3 pad 19: SW_5 -> SW_8
- U3 pad 20: SW_2 -> SW_1
- U3 pad 42: SW_7 -> SW_5
- U3 pad 43: SW_10 -> SW_2
- U3 pad 45: SW_9 -> SW_7
- U3 pad 46: SW_8 -> unconnected-(U3-Pad46)
Routing:
- net +3.3VA: track 0.00 -> 91.5 mm, vias 0 -> 6
- net +5V: track 0.00 -> 77.1 mm, vias 0 -> 4
- net SW_9: track 0.00 -> 72.5 mm, vias 0 -> 1
- net /D1+: track 3.93 -> 67.4 mm, vias 0 -> 4
- net /D1-: track 3.91 -> 63.3 mm, vias 0 -> 3
- net SW_7: track 0.00 -> 57.1 mm, vias 0 -> 1
- net SW_2: track 0.00 -> 44.7 mm
- net SW_3: track 0.00 -> 41.4 mm, vias 0 -> 1
- net SW_5: track 0.00 -> 40.6 mm
- net SW_8: track 0.00 -> 39.5 mm, vias 0 -> 1
- net SW_10: track 0.00 -> 38.1 mm, vias 0 -> 1
- net /BOOT: track 0.00 -> 27.9 mm, vias 0 -> 2
- net SW_6: track 0.00 -> 20.1 mm
- net SW_4: track 0.00 -> 18.3 mm
- net SW_1: track 0.00 -> 12.7 mm
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Other:
- board outline added: 109.5 x 109.5 mm
