File: PCB/herringbone_macro_pad.kicad_sch (KiCad schematic)
At the start: 11 parts, among them SW1 CherryMX_2.75u_PCB_StabWireBo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, SW10 CherryMX_1.00u_PCB, SW2 CherryMX_1.00u_PCB, SW3 CherryMX_2.75u_PCB_StabWireBo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, SW4 CherryMX_2.75u_PCB_StabWireBo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, SW5 CherryMX_1.00u_PCB, SW6 CherryMX_2.75u_PCB_StabWireBo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, SW7 CherryMX_2.75u_PCB_StabWireBo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, SW8 CherryMX_1.00u_PCB, SW9 CherryMX_2.75u_PCB_StabWireBo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, U1 RP2040

Commit message: update, hardware rev 2.0
Parts:
- removed U1: RP2040, herringbone_macro_pad:Seeeduino XIAO-MOUDLE14P-2.54-21X17.8MM, symbol Seeeduino XIAO:SeeeduinoXIAO
- added C1, C2: 22p, Keebio-Parts:C_0603, symbol Device:C_Small
- added C10: 10n, Keebio-Parts:C_0603, symbol Device:C_Small
- added C11: 1u, Keebio-Parts:C_0603, symbol Device:C_Small
- added C12: 0.1u, Keebio-Parts:C_0603, symbol Device:C_Small
- added C3: 22u, Keebio-Parts:C_0603, symbol Device:C_Small
- added C4: 10u, Keebio-Parts:C_0603, symbol Device:C_Small
- added C5: 4.7u, Keebio-Parts:C_0603, symbol Device:C_Small
- added C6, C7, C8, C9: 100n, Keebio-Parts:C_0603, symbol Device:C_Small
- added D1: D_Small, Keebio-Parts:D_0805, symbol Device:D_Small
- added J1: Screw_Terminal_01x04, Connector_JST:JST_SH_SM04B-SRSS-TB_1x04-1MP_P1.00mm_Horizontal, symbol Connector:Screw_Terminal_01x04
- added R1, R2: 5.1k, Keebio-Parts:R_0603, symbol Device:R_Small_US
- added R5: 10k, Keebio-Parts:R_0603, symbol Device:R_Small_US
- added SW11: SW_Push, Keebio-Parts:SW_SPST_TL3342, symbol Switch:SW_Push
- added U1: SRV05-4, Package_TO_SOT_SMD:SOT-23-6, symbol Power_Protection:SRV05-4
- added U2: AMS1117, Package_TO_SOT_SMD:SOT-223-3_TabPin2, symbol Regulator_Linear:AMS1117
- added U3: STM32L151C8TxA, Package_QFP:LQFP-48_7x7mm_P0.5mm, symbol MCU_ST_STM32L1:STM32L151C8TxA
- added USB1: C167321, Keebio-Parts:HRO-TYPE-C-31-M-12-Assembly, symbol keebio:HRO-TYPE-C-31-M-12
- added Y1: Crystal, Crystal:Crystal_SMD_0603-2Pin_6.0x3.5mm, symbol Device:Crystal
Connections:
- net GND: now also C1.1, C10.2, C11.2, C12.2, C2.2, C3.2, C4.2, C5.2, C6.2, C7.2, C8.2, C9.2, J1.1 (Pin_1), R1.1, R2.1, SW11.2, U1.2 (VN), U3.23 (VSS), U3.35 (VSS), U3.47 (VSS), U3.8 (VSSA), USB1.1 (GND), USB1.12 (GND), USB1.13 (SHIELD)
- net SW_0: now also U3.20 (PB2)
- net SW_1: now also U3.22 (PB11)
- net SW_2: now also U3.17 (PA7)
- net SW_3: now also U3.18 (PB0)
- net SW_4: now also U3.38 (PA15)
- net SW_5: now also U3.21 (PB10)
- net SW_6: now also U3.19 (PB1)
- net SW_7: now also U3.37 (PA14)
- net SW_8: now also U3.40 (PB4)
- net SW_9: now also U3.39 (PB3)
- new net: R2.2, USB1.10 (CC2)
- new net: R1.2, USB1.4 (CC1)
- new net: C4.1, U2.1 (ADJ)
- new net +3.3VA: C10.1, C11.1, C5.1, C6.1, C7.1, C8.1, C9.1, D1.2 (A), R5.1, U2.2 (VO), U3.24 (VDD), U3.36 (VDD), U3.48 (VDD), U3.9 (VDDA)
- new net +5V: C3.1, D1.1 (K), J1.4 (Pin_4), U1.5 (VP), U2.3 (VI), USB1.11 (VBUS), USB1.2 (VBUS)
- new net CLK_IN: C1.2, U3.5 (PH0), Y1.2
- new net CLK_OUT: C2.1, U3.6 (PH1), Y1.1
- new net D1+: J1.2 (Pin_2), U1.1 (IO1), U1.4 (IO3), U3.33 (PA12), USB1.6 (DP1), USB1.8 (DP2)
- new net D1-: J1.3 (Pin_3), U1.3 (IO2), U1.6 (IO4), U3.32 (PA11), USB1.5 (DN2), USB1.7 (DN1)
- new net RST: C12.1, R5.2, SW11.1, U3.7 (NRST)
- no-connect marks 9 -> 2

Commit message: Hardware revision.
Parts:
- removed C11: 1u, Keebio-Parts:C_0603, symbol Device:C_Small
- removed R5: 10k, Keebio-Parts:R_0603, symbol Device:R_Small_US
- removed SW1, SW3, SW4, SW6, SW7, SW9: CherryMX_2.75u_PCB_StabWireBottom, CherryMX_PCB_StabWireBottom:CherryMX_2.75u_PCB_StabWireBottom, symbol Switch:SW_Push
- removed SW10, SW2, SW5, SW8: CherryMX_1.00u_PCB, CherryMX_PCB:CherryMX_1.00u_PCB, symbol Switch:SW_Push
- removed U3: STM32L151C8TxA, Package_QFP:LQFP-48_7x7mm_P0.5mm, symbol MCU_ST_STM32L1:STM32L151C8TxA
- added C13, C14: 0.1u, Keebio-Parts:C_0402, symbol Device:C_Small
- added C3, C4: 4.7u, Keebio-Parts:C_0402, symbol Device:C_Small
- added R3: 10k, Keebio-Parts:R_0402, symbol Device:R_Small_US
- added SW2: SW_SPST, Button_Switch_SMD:SW_SPDT_PCM12, symbol Switch:SW_SPST
- added U3: STM32F411CEUx, Package_DFN_QFN:QFN-48-1EP_7x7mm_P0.5mm_EP5.6x5.6mm, symbol MCU_ST_STM32F4:STM32F411CEUx
- C1: renamed from C3; footprint Keebio-Parts:C_0603 -> Keebio-Parts:C_0402
- C10: value 10n -> 0.1u; footprint Keebio-Parts:C_0603 -> Keebio-Parts:C_0402
- C11: renamed from C1; value 22p -> 30p; footprint Keebio-Parts:C_0603 -> Keebio-Parts:C_0402
- C12: renamed from C2; value 22p -> 30p; footprint Keebio-Parts:C_0603 -> Keebio-Parts:C_0402
- C15: renamed from C12; footprint Keebio-Parts:C_0603 -> Keebio-Parts:C_0402
- C2: renamed from C4; footprint Keebio-Parts:C_0603 -> Keebio-Parts:C_0402
- C5: value 4.7u -> 0.1u; footprint Keebio-Parts:C_0603 -> Keebio-Parts:C_0402
- C6, C7, C9: value 100n -> 0.1u; footprint Keebio-Parts:C_0603 -> Keebio-Parts:C_0402
- C8: value 100n -> 4.7u; footprint Keebio-Parts:C_0603 -> Keebio-Parts:C_0402
- J1: value Screw_Terminal_01x04 -> JST
- R1, R2: footprint Keebio-Parts:R_0603 -> Keebio-Parts:R_0402
- renumbered SW11 to SW1
Connections:
- net +3.3VA: now also C13.1, C14.1, C3.1, C4.1, U3.24 (VDD), U3.36 (VDD), U3.48 (VDD), U3.9 (VDDA); no longer C8.1
- net CLK_IN: now also U3.5 (PH0)
- net CLK_OUT: now also U3.6 (PH1)
- net D1+: now also U3.33 (PA12)
- net D1-: now also U3.32 (PA11)
- net GND: now also C13.2, C14.2, C3.2, C4.2, R3.1, U3.23 (VSS), U3.35 (VSS), U3.47 (VSS), U3.49 (VSS), U3.8 (VSSA)
- net RST: now also U3.7 (NRST)
- net SW_1: now also U3.18 (PB0)
- net SW_2: now also U3.20 (PB2)
- net SW_3: now also U3.40 (PB4)
- net SW_4: now also U3.39 (PB3)
- net SW_5: now also U3.19 (PB1)
- net SW_6: now also U3.41 (PB5)
- net SW_7: now also U3.42 (PB6)
- net SW_8: now also U3.46 (PB9)
- net SW_9: now also U3.45 (PB8)
- new net: R3.2, SW2.1 (A)
- new net BOOT: SW2.2 (B), U3.44 (BOOT0)
- new net SW_10: U3.43 (PB7)
- new net V_CAP: C8.1, U3.22 (VCAP1)
- no-connect marks 2 -> 3
Other:
- added sheet SW_MATRIX (untitled.kicad_sch)
- note added: "Power Conditioning"
- note added: "Reset/Boot"
- moved on the sheet: C1, C11, C12, C15, C2, D1, J1, R1, R2, SW1, U1, U2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

Commit message: Hardware revision 2/17/2022
Parts:
- added D2: LED, Diode_SMD:D_0402_1005Metric, symbol Device:LED
- added R4: 370, Keebio-Parts:R_0402, symbol Device:R_Small_US
Connections:
- net +3.3VA: now also C1.1, R4.1
- net +5V: no longer C1.1
- net GND: now also D2.1 (K)
- net SW_1: now also U3.20 (PB2); no longer U3.18 (PB0)
- net SW_10: now also U3.17 (PA7); no longer U3.43 (PB7)
- net SW_2: now also U3.43 (PB7); no longer U3.20 (PB2)
- net SW_5: now also U3.42 (PB6); no longer U3.19 (PB1)
- net SW_7: now also U3.45 (PB8); no longer U3.42 (PB6)
- net SW_8: now also U3.19 (PB1); no longer U3.46 (PB9)
- net SW_9: now also U3.18 (PB0); no longer U3.45 (PB8)
- new net: D2.2 (A), R4.2
Other:
- moved on the sheet: C1
